File: PCB/thrfv.kicad_pcb (KiCad board)
At the start: 2 copper layers, 126.3 x 98.6 mm, 84 parts, among them J1 4PIN, J2 OLED, J3 Conn_01x05_Female, J4 Conn_01x05_Female, SW1 SW1, SW10 SW10, SW11 SW11, SW12 SW12, SW13 SW13, SW14 SW14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

Commit message: Minor changes here and there.
Parts:
- U1: footprint jw_custom_footprint:ProMicro_jumper_pad_only_zigzag -> jw_custom_footprint:ProMicro_jumper_pad_only
- moved D16 1.25 mm to (135.2, 130.5)
- moved D17 1.16 mm to (150.8, 130.5)
- moved D1 0.50 mm to (116.0, 76.3)
- moved D6 0.50 mm to (116.0, 95.3)
- moved SW1 0.50 mm to (107.9, 74.5)
- moved SW11 0.50 mm to (107.9, 112.5)
- moved SW6 0.50 mm to (107.9, 93.5)
- moved D11 0.50 mm to (116.0, 114.4)
- moved JY_BT_1 0.50 mm to (123.7, 123.7)
- moved TH3 0.50 mm to (114.5, 123.7)
- moved TH2 0.41 mm to (115.8, 63.4)
- moved SW5 0.05 mm to (183.9, 73.5)
- moved D5 0.05 mm to (192.0, 75.3)
Routing:
- net row3: track 96.5 -> 94.9 mm
- net Net-(D16-Pad2): track 2.67 -> 3.88 mm
- net col4: track 116.9 -> 115.7 mm
- net Net-(D17-Pad2): track 2.76 -> 3.83 mm
- net Net-(D18-Pad2): track 8.29 -> 9.22 mm
- net row0: track 109.3 -> 110.1 mm
- net ENCA: track 86.4 -> 85.7 mm
Other:
- outline, holes or cut-outs redrawn

Commit message: No comment.
Parts:
- removed the REF** at (199.1, 69.6)
- removed the REF** at (210.1, 69.6)
- removed the REF** at (145.9, 129.2) (x2)
- added REF**: Nintendo_Switch_JOYSTICK, jw_custom_footprint:Nintendo_Switch_JOYSTICK, F.Cu at (146.1, 129.5)
- added REF**: Nintendo_Switch_JOYSTICK, jw_custom_footprint:Nintendo_Switch_JOYSTICK, B.Cu at (146.1, 129.5)
- J3, J4: footprint jw_custom_footprint:Molex_200528-0050_1x05-1MP_P0.5mm_Horizontal -> Connector_FFC-FPC:TE_0-1734839-5_1x05-1MP_P0.5mm_Horizontal
- moved JY_BT_1 6.88 mm to (122.3, 130.4)
- moved TH3 5.78 mm to (119.3, 120.4)
- moved SW17 0.75 mm to (146.1, 130.4)
- moved SW16 0.75 mm to (130.5, 130.4)
- moved D4 0.55 mm to (172.9, 73.1)
- moved D8 0.51 mm to (153.9, 89.6)
- moved D13 0.44 mm to (153.9, 108.6)
- moved D3 0.44 mm to (153.9, 70.6)
- moved D9 0.43 mm to (172.9, 92.1)
- moved D2 0.43 mm to (134.9, 73.1)
- moved D5 0.39 mm to (191.9, 75.7)
- moved D14 0.38 mm to (172.9, 111.1)
- moved D7 0.35 mm to (134.9, 92.1)
- moved D15 0.34 mm to (191.9, 113.7)
- moved D1 0.33 mm to (115.9, 76.6)
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Routing:
- net Net-(D8-Pad2): track 3.42 -> 5.21 mm
- net Net-(D4-Pad2): track 3.42 -> 5.21 mm
- net Net-(D13-Pad2): track 3.34 -> 5.06 mm
- net Net-(D9-Pad2): track 3.39 -> 5.06 mm
- net Net-(D5-Pad2): track 3.85 -> 5.49 mm
- net Net-(D14-Pad2): track 3.44 -> 5.06 mm
- net Net-(D2-Pad2): track 3.66 -> 5.28 mm
- net Net-(D15-Pad2): track 3.61 -> 5.21 mm
- net Net-(D1-Pad2): track 3.71 -> 5.28 mm
- net Net-(D6-Pad2): track 3.64 -> 5.21 mm
- net Net-(D10-Pad2): track 3.66 -> 5.21 mm
- net Net-(D7-Pad2): track 3.52 -> 5.06 mm
- net Net-(D11-Pad2): track 3.62 -> 5.14 mm
- net Net-(D12-Pad2): track 3.65 -> 5.06 mm
- net Net-(J1-Pad2): track 34.2 -> 35.6 mm
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Other:
- outline, holes or cut-outs redrawn
- board text removed: "Pro_Micro_Type-C_Extension"

Commit message: No comment.
Parts:
- moved D3 2.54 mm to (153.9, 68.1)
- moved D8 2.54 mm to (153.9, 87.1)
- moved SW13 2.54 mm to (146.1, 104.2)
- moved D13 2.54 mm to (153.9, 106.1)
- moved LED3 2.54 mm to (147.8, 93.1)
- moved SW3 2.54 mm to (146.1, 66.2)
- moved SW8 2.54 mm to (146.1, 85.2)
- moved RSW1 2.31 mm to (185.9, 59.6)
- moved RSW2 2.31 mm to (185.9, 59.6)
- moved D1 1.96 mm to (115.9, 74.7)
- moved D11 1.96 mm to (115.9, 112.7)
- moved D6 1.96 mm to (115.9, 93.7)
- moved TH2 1.96 mm to (116.0, 61.7)
- moved SW1 1.96 mm to (108.1, 72.8)
- moved SW11 1.96 mm to (108.1, 110.8)
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Routing:
- net row3: track 96.0 -> 103.3 mm, vias 3 -> 4
- net RST: track 38.4 -> 40.6 mm
- net col1: track 187.6 -> 189.8 mm
- net col0: track 204.2 -> 206.3 mm
- net Axis_X: track 110.9 -> 109.0 mm
- net Axis_Y: track 108.1 -> 106.3 mm
- net col4: track 116.0 -> 117.8 mm
- net BT: track 108.6 -> 107.0 mm
- net col2: track 176.1 -> 177.5 mm
- net col3: track 148.7 -> 150.1 mm
- net row2: track 110.3 -> 111.6 mm
- net row0: track 109.3 -> 110.6 mm
- net row1: track 100.6 -> 101.9 mm
- net VCC: track 235.4 -> 236.5 mm
- net Net-(LED3-Pad2): track 37.8 -> 38.5 mm
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Other:
- board size 126.3 x 98.6 mm -> 126.3 x 101 mm

Commit message: Multiple changes. Re-plotted gerber files.
Parts:
- moved RSW1 0.84 mm to (185.9, 60.4)
- moved RSW2 0.84 mm to (185.9, 60.4)
- moved D12 0.81 mm to (134.9, 110.7)
- moved D2 0.81 mm to (134.9, 72.7)
- moved D3 0.81 mm to (153.9, 68.9)
- moved D7 0.81 mm to (134.9, 91.7)
- moved D8 0.81 mm to (153.9, 87.9)
- moved D9 0.81 mm to (172.9, 91.7)
- moved J3 0.81 mm to (132.4, 125.2)
- moved J4 0.81 mm to (159.8, 125.2)
- moved JS_HOLE_1 0.81 mm to (153.2, 118.3)
- moved JS_HOLE_2 0.81 mm to (139.1, 118.3)
- moved JY_CABLE_1 0.81 mm to (132.4, 117.9)
- moved JY_CABLE_2 0.81 mm to (159.8, 117.9)
- moved LED4 0.81 mm to (122.9, 98.7)
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Connections:
- EC1 pad MP: (no net) -> col4
Routing:
- net row3: track 103.3 -> 98.1 mm, vias 4 -> 3
- net GND: track 20.6 -> 21.6 mm, vias 20 -> 17
- net Axis_Y: track 106.3 -> 107.1 mm
- net BT: track 107.0 -> 107.8 mm
- net Axis_X: track 109.0 -> 109.8 mm
- net row2: track 111.6 -> 111.0 mm
- net col3: track 150.1 -> 149.4 mm
- net row1: track 101.9 -> 101.2 mm
- net row0: track 110.6 -> 109.9 mm
- net col0: track 206.3 -> 205.6 mm
- net ENCB: track 90.7 -> 91.3 mm
Other:
- board size 126.3 x 101 mm -> 126.3 x 100.1 mm

Commit message: First PCB production.
Parts:
- JY_CABLE_1, JY_CABLE_2: footprint jw_custom_footprint:Mounting_Hole_7x3mm -> jw_custom_footprint:Mounting_Hole_6.5x2.54mm
- moved D16 17.9 mm to (153.0, 127.3), turned to 180 degrees
- moved D17 2.05 mm to (153.0, 130.0), turned to 180 degrees
- moved JY_BT_2 1.35 mm to (160.5, 130.1)
- moved JS_HOLE_1 1.31 mm to (153.2, 117.0)
- moved JS_HOLE_2 1.31 mm to (139.1, 117.0)
- moved JY_CABLE_1 0.93 mm to (132.4, 117.0)
- moved JY_CABLE_2 0.93 mm to (159.8, 117.0)
- moved JS_HOLE_3 0.51 mm to (136.7, 134.9)
- moved JS_HOLE_4 0.51 mm to (155.6, 134.9)
- moved REF** 0.51 mm to (146.1, 127.9) (x2)
- moved J3 0.31 mm to (132.4, 124.9)
- moved J4 0.31 mm to (159.8, 124.9)
- moved JY_BT_1 0.24 mm to (122.3, 130.1)
- moved SW16 0.24 mm to (130.5, 130.1)
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Connections:
- EC1 pad MP: col4 -> (no net)
Routing:
- net row3: track 98.1 -> 78.0 mm
- net Net-(D16-Pad2): track 4.08 -> 20.5 mm
- net VCC: track 236.5 -> 239.1 mm
- net Axis_Y: track 107.1 -> 104.8 mm
- net Net-(J1-Pad2): track 35.6 -> 33.9 mm
- net col4: track 117.8 -> 116.5 mm
- net BT: track 107.8 -> 106.7 mm
- net col3: track 149.4 -> 148.3 mm
- net Axis_X: track 109.8 -> 108.7 mm
- net RST: track 40.6 -> 39.8 mm
- net SDA: track 49.1 -> 48.3 mm
- net col2: track 177.1 -> 176.5 mm
- net sw_row: track 36.9 -> 36.3 mm
- net GND: track 21.6 -> 21.1 mm, vias 17 -> 15
- net col1: track 189.4 -> 188.9 mm
