File: PCB/thrfv.kicad_pcb (KiCad board)
At the start: 2 copper layers, 126.3 x 100.1 mm, 82 parts, among them J1 4PIN, J2 OLED, J3 Conn_01x05_Female, J4 Conn_01x05_Female, SW1 SW1, SW10 SW10, SW11 SW11, SW12 SW12, SW13 SW13, SW14 SW14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

Commit message: No comment.
Parts:
- EC1: footprint jw_custom_footprint:RotaryEncoder_Alps_EC11E-Switch_Vertical_H20mm -> jw_custom_footprint:RotaryEncoder_Alps_EC11E-Switch_Vertical_H20mm_no_copper_MP
- J3, J4: footprint Connector_FFC-FPC:TE_0-1734839-5_1x05-1MP_P0.5mm_Horizontal -> jw_custom_footprint:FPC_front_flip_connector_1x05-P0.5mm_Horizontal
- JY_CABLE_1: footprint jw_custom_footprint:Mounting_Hole_6.5x2.54mm -> jw_custom_footprint:Nintendo_Switch_Joystick_Cable_Hole_6x2mm
- JY_CABLE_2: footprint jw_custom_footprint:Mounting_Hole_6.5x2.54mm -> jw_custom_footprint:Nintendo_Switch_Joystick_Cable_Hole_5.5x2mm
- moved D16 15.9 mm to (137.3, 130.1)
- moved J3 1.98 mm to (133.9, 123.6), turned to 0 degrees
- moved J4 1.98 mm to (158.4, 123.6), turned to 180 degrees
- moved JY_CABLE_1 1.46 mm to (133.9, 116.8)
- moved JY_CABLE_2 1.46 mm to (158.4, 116.8)
- moved D17 1.30 mm to (154.3, 130.1)
- moved D20 0.50 mm to (191.1, 124.3)
- moved D19 0.36 mm to (188.3, 124.3)
- moved D18 0.23 mm to (185.5, 124.3)
Routing:
- net Net-(D16-Pad2): track 20.5 -> 3.73 mm
- net row3: track 78.0 -> 93.2 mm
- net Net-(D19-Pad2): track 20.2 -> 18.3 mm
- net Axis_X: track 108.7 -> 106.9 mm
- net BT: track 106.7 -> 104.9 mm
- net Axis_Y: track 104.8 -> 103.1 mm
- net VCC: track 239.1 -> 240.3 mm
- net sw_row: track 36.3 -> 37.3 mm
- net Net-(D17-Pad2): track 3.76 -> 4.76 mm
- net ENCB: track 90.8 -> 90.1 mm
- net ENCA: track 86.4 -> 85.7 mm
- net GND: track 21.1 -> 20.4 mm
