File: PCB/thrfv.kicad_sch (KiCad schematic)
At the start: 80 parts, among them J1 4PIN, J2 OLED, J3 Conn_01x05_Female, J4 Conn_01x05_Female, SW1 SW1, SW10 SW10, SW11 SW11, SW12 SW12, SW13 SW13, SW14 SW14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

Commit message: 1. Repository renamed from AT_ST to thrfv, aka three-by-five, 3x5 2. Multiple twists.
Parts:
- SW16: footprint jw_custom_footprint:contact_button_pad_death_star_5mm_dual_side -> jw_custom_footprint:contact_button_pad_half_circle_3mm
- SW17: footprint jw_custom_footprint:contact_button_pad_planet_5mm_dual_side -> jw_custom_footprint:contact_button_pad_half_circle_3mm
- U1: footprint jw_custom_footprint:ProMicro_jumper_pad_only -> jw_custom_footprint:ProMicro_jumper_pad_only_zigzag
Changed lines of the file:
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@@
       (effects (font (size 1.524 1.524)))
     )
-    (property "Footprint" "jw_custom_footprint:ProMicro_jumper_pad_only" (id 2) (at 102.108 58.674 0)
+    (property "Footprint" "jw_custom_footprint:ProMicro_jumper_pad_only_zigzag" (id 2) (at 102.108 58.674 0)
       (effects (font (size 1.524 1.524)) hide)
     )
@@
     (property "Reference" "SW17" (id 0) (at 186.436 83.693 0))
     (property "Value" "SW_Contact_Pad" (id 1) (at 188.087 86.741 0))
-    (property "Footprint" "jw_custom_footprint:contact_button_pad_planet_5mm_dual_side" (id 2) (at 191.516 83.312 0)
+    (property "Footprint" "jw_custom_footprint:contact_button_pad_half_circle_3mm" (id 2) (at 191.516 83.312 0)
       (effects (font (size 1.27 1.27)) hide)
     )
@@
     (property "Reference" "SW16" (id 0) (at 165.735 83.947 0))
     (property "Value" "SW_Contact_Pad" (id 1) (at 167.64 86.741 0))
-    (property "Footprint" "jw_custom_footprint:contact_button_pad_death_star_5mm_dual_side" (id 2) (at 171.069 83.312 0)
+    (property "Footprint" "jw_custom_footprint:contact_button_pad_half_circle_3mm" (id 2) (at 171.069 83.312 0)
       (effects (font (size 1.27 1.27)) hide)
     )
@@
     )
     (path "/ddf50807-8c6e-4139-bb13-aa0ef1274689"
-      (reference "SW16") (unit 1) (value "SW_Contact_Pad") (footprint "jw_custom_footprint:contact_button_pad_death_star_5mm_dual_side")
+      (reference "SW16") (unit 1) (value "SW_Contact_Pad") (footprint "jw_custom_footprint:contact_button_pad_half_circle_3mm")
     )
     (path "/34e04860-0169-4bbd-8058-25fde9672465"
-      (reference "SW17") (unit 1) (value "SW_Contact_Pad") (footprint "jw_custom_footprint:contact_button_pad_planet_5mm_dual_side")
+      (reference "SW17") (unit 1) (value "SW_Contact_Pad") (footprint "jw_custom_footprint:contact_button_pad_half_circle_3mm")
     )
     (path "/c6a23e69-6689-4411-b957-a6d23f8db0db"
@@
     )
     (path "/00000000-0000-0000-0000-00005b722440"
-      (reference "U1") (unit 1) (value "ProMicro") (footprint "jw_custom_footprint:ProMicro_jumper_pad_only")
-    )
-  )
+      (reference "U1") (unit 1) (value "ProMicro") (footprint "jw_custom_footprint:ProMicro_jumper_pad_only_zigzag")
+    )
+  )

Commit message: Minor changes here and there.
Parts:
- U1: footprint jw_custom_footprint:ProMicro_jumper_pad_only_zigzag -> jw_custom_footprint:ProMicro_jumper_pad_only
Changed lines of the file:
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@@
       (effects (font (size 1.524 1.524)))
     )
-    (property "Footprint" "jw_custom_footprint:ProMicro_jumper_pad_only_zigzag" (id 2) (at 102.108 58.674 0)
+    (property "Footprint" "jw_custom_footprint:ProMicro_jumper_pad_only" (id 2) (at 102.108 58.674 0)
       (effects (font (size 1.524 1.524)) hide)
     )
@@
     )
     (path "/00000000-0000-0000-0000-00005b722440"
-      (reference "U1") (unit 1) (value "ProMicro") (footprint "jw_custom_footprint:ProMicro_jumper_pad_only_zigzag")
-    )
-  )
+      (reference "U1") (unit 1) (value "ProMicro") (footprint "jw_custom_footprint:ProMicro_jumper_pad_only")
+    )
+  )

Commit message: No comment.
Parts:
- J3, J4: footprint jw_custom_footprint:Molex_200528-0050_1x05-1MP_P0.5mm_Horizontal -> Connector_FFC-FPC:TE_0-1734839-5_1x05-1MP_P0.5mm_Horizontal
Changed lines of the file:
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@@
       (effects (font (size 1.27 1.27)) (justify left))
     )
-    (property "Footprint" "jw_custom_footprint:Molex_200528-0050_1x05-1MP_P0.5mm_Horizontal" (id 2) (at 238.76 121.92 0)
+    (property "Footprint" "Connector_FFC-FPC:TE_0-1734839-5_1x05-1MP_P0.5mm_Horizontal" (id 2) (at 238.76 121.92 0)
       (effects (font (size 1.27 1.27)) hide)
     )
@@
       (effects (font (size 1.27 1.27)) (justify left))
     )
-    (property "Footprint" "jw_custom_footprint:Molex_200528-0050_1x05-1MP_P0.5mm_Horizontal" (id 2) (at 213.36 121.92 0)
+    (property "Footprint" "Connector_FFC-FPC:TE_0-1734839-5_1x05-1MP_P0.5mm_Horizontal" (id 2) (at 213.36 121.92 0)
       (effects (font (size 1.27 1.27)) hide)
     )
@@
     )
     (path "/33de51e4-f43b-45b1-833b-e21d84d90255"
-      (reference "J3") (unit 1) (value "Conn_01x05_Female") (footprint "jw_custom_footprint:Molex_200528-0050_1x05-1MP_P0.5mm_Horizontal")
+      (reference "J3") (unit 1) (value "Conn_01x05_Female") (footprint "Connector_FFC-FPC:TE_0-1734839-5_1x05-1MP_P0.5mm_Horizontal")
     )
     (path "/2eec7e7a-4330-4f6e-9016-3a7281b4315e"
-      (reference "J4") (unit 1) (value "Conn_01x05_Female") (footprint "jw_custom_footprint:Molex_200528-0050_1x05-1MP_P0.5mm_Horizontal")
+      (reference "J4") (unit 1) (value "Conn_01x05_Female") (footprint "Connector_FFC-FPC:TE_0-1734839-5_1x05-1MP_P0.5mm_Horizontal")
     )
     (path "/00000000-0000-0000-0000-00005b913c11"
